Commit message: Body of the robot is now similar to actual robot, also spawn.launch edited to puvklish tf values, lidar also works for the simulation

File: ros_ws/src/kamu_robotu/kamu_robotu_gazebo/urdf/kamu_robotu.xacro (robot description, xacro)
@@ -1,10 +1,10 @@
 <?xml version="1.0"?>
 <robot name="kamu_robotu" xmlns:xacro="https://www.ros.org/wiki/xacro" >
-  <!--<xacro:include filename="$(find kamu_robotu_gazebo)/urdf/kamu_robotu.gazebo.xacro"/> -->
-  <xacro:arg name="laser_visual" default="true"/>
-  <xacro:arg name="imu_visual"   default="true"/>
+  <xacro:arg name="laser_visual" default="false"/>
+  <xacro:arg name="imu_visual"   default="false"/>
   <xacro:property name="wheel_radius" value="0.024" />
   <xacro:property name="wheel_length" value="0.01" />
   <xacro:property name="wheel_seperation" value="0.2" />
+  <xacro:property name="chasis_height" value="0.115" />
   <material name="black">
     <color rgba="0.0 0.0 0.0 1.0"/>
@@ -31,14 +31,14 @@
     <color rgba="1.0 1.0 1.0 1.0"/>
   </material>
-  <gazebo reference="link_chassis">
+  <gazebo reference="base_link">
     <material>Gazebo/Orange</material>
   </gazebo>
-  <gazebo reference="link_left_wheel">
+  <gazebo reference="wheel_left_link">
     <material>Gazebo/Blue</material>
   </gazebo>
-  <gazebo reference="link_right_wheel">
+  <gazebo reference="wheel_right_link">
     <material>Gazebo/Blue</material>
   </gazebo>
-  <link name="link_chassis">
+  <link name="base_link">
     <!-- pose and inertial -->
     <pose>0 0 0.1 0 0 0</pose>
@@ -50,11 +50,12 @@
     <collision name="collision_chassis">
       <geometry>
-        <box size="0.18 0.18 0.005"/>
+        <cylinder length="0.015" radius="0.2"/>
       </geometry>
     </collision>
     <visual>
+      <pose>0 0 0 0 1.57080 1.5708</pose>
       <origin rpy="0 0 0" xyz="0 0 0"/>
       <geometry>
-        <box size="0.18 0.18 0.005"/>
+        <mesh filename="package://kamu_robotu_gazebo/meshes/base.STL" scale="1 1 1"/>
       </geometry>
       <material name="blue"/>
@@ -62,7 +63,7 @@
     <!-- caster front -->
     <collision name="caster_front_collision">
-      <origin rpy=" 0 0 0" xyz="0.05 0 0"/>
-      <geometry>
-        <sphere radius="0.0235"/>
+      <origin rpy=" 0 0 0" xyz="0.05 0 -${chasis_height/2}"/>
+      <geometry>
+        <sphere radius="0.0239"/>
       </geometry>
       <surface>
@@ -78,14 +79,14 @@
     </collision>
     <visual name="caster_front_visual">
-      <origin rpy=" 0 0 0" xyz="0.05 0 0"/>
-      <geometry>
-        <sphere radius="0.0235"/>
+      <origin rpy=" 0 0 0" xyz="0.05 0 -${chasis_height/2}"/>
+      <geometry>
+        <sphere radius="0.0239"/>
       </geometry>
     </visual>
     <!-- caster back -->
     <collision name="caster_back_collision">
-      <origin rpy=" 0 0 0" xyz="-0.05 0 0"/>
-      <geometry>
-        <sphere radius="0.0235"/>
+      <origin rpy=" 0 0 0" xyz="-0.05 0 -${chasis_height/2}"/>
+      <geometry>
+        <sphere radius="0.0238"/>
       </geometry>
       <surface>
@@ -101,12 +102,12 @@
     </collision>
     <visual name="caster_back_visual">
-      <origin rpy=" 0 0 0" xyz="-0.05 0 0"/>
-      <geometry>
-        <sphere radius="0.0235"/>
-      </geometry>
-    </visual>
+      <origin rpy=" 0 0 0" xyz="-0.05 0 -${chasis_height/2}"/>
+      <geometry>
+        <sphere radius="0.0239"/>
+      </geometry>
+    </visual>
+  </link>
   <!-- Create wheel right -->
-  </link>
-  <link name="link_right_wheel">
+  <link name="wheel_right_link">
     <inertial>
       <mass value="0.2"/>
@@ -114,5 +115,5 @@
       <inertia ixx="0.00052666666" ixy="0" ixz="0" iyy="0.00052666666" iyz="0" izz="0.001"/>
     </inertial>
-    <collision name="link_right_wheel_collision">
+    <collision name="wheel_right_link_collision">
       <origin rpy="0 1.5707 1.5707" xyz="0 0 0" />
       <geometry>
@@ -120,5 +121,5 @@
       </geometry>
     </collision>
-    <visual name="link_right_wheel_visual">
+    <visual name="wheel_right_link_visual">
       <origin rpy="0 1.5707 1.5707" xyz="0 0 0"/>
       <geometry>
@@ -127,15 +128,6 @@
     </visual>
   </link>
-  <!--   Joint for right wheel  -->
-  <joint name="joint_right_wheel" type="continuous">
-    <origin rpy="0 0 0" xyz="0 ${wheel_seperation/2} 0"/>
-    <child link="link_right_wheel" />
-    <parent link="link_chassis"/>
-    <axis rpy="0 0 0" xyz="0 1 0"/>
-    <limit effort="10000" velocity="1000"/>
-    <joint_properties damping="1.0" friction="1.0" />
-  </joint>
   <!-- Left Wheel link -->
-  <link name="link_left_wheel">
+  <link name="wheel_left_link">
     <inertial>
       <mass value="0.2"/>
@@ -143,5 +135,5 @@
       <inertia ixx="0.00052666666" ixy="0" ixz="0" iyy="0.00052666666" iyz="0" izz="0.001"/>
     </inertial>
-    <collision name="link_left_wheel_collision">
+    <collision name="wheel_left_link_collision">
       <origin rpy="0 1.5707 1.5707" xyz="0 0 0" />
       <geometry>
@@ -149,5 +141,5 @@
       </geometry>
     </collision>
-    <visual name="link_left_wheel_visual">
+    <visual name="wheel_left_link_visual">
       <origin rpy="0 1.5707 1.5707" xyz="0 0 0"/>
       <geometry>
@@ -157,8 +149,17 @@
   </link>
   <!--   Joint for right wheel  -->
-  <joint name="joint_left_wheel" type="continuous">
-    <origin rpy="0 0 0" xyz="0 -${wheel_seperation/2} 0"/>
-    <child link="link_left_wheel" />
-    <parent link="link_chassis"/>
+  <joint name="wheel_right_joint" type="continuous">
+    <origin rpy="0 0 0" xyz="0 ${wheel_seperation/2} -${chasis_height/2}"/>
+    <child link="wheel_right_link" />
+    <parent link="base_link"/>
+    <axis rpy="0 0 0" xyz="0 1 0"/>
+    <limit effort="10000" velocity="1000"/>
+    <joint_properties damping="1.0" friction="1.0" />
+  </joint>
+  <!--   Joint for left wheel  -->
+  <joint name="wheel_left_joint" type="continuous">
+    <origin rpy="0 0 0" xyz="0 -${wheel_seperation/2} -${chasis_height/2}"/>
+    <child link="wheel_left_link" />
+    <parent link="base_link"/>
     <axis rpy="0 0 0" xyz="0 1 0"/>
     <limit effort="10000" velocity="1000"/>
@@ -166,13 +167,13 @@
   </joint>
   <joint name="imu_joint" type="fixed">
-    <parent link="link_chassis"/>
+    <parent link="base_link"/>
     <child link="imu_link"/>
-    <origin xyz="-0.032 0 0.068" rpy="0 0 0"/>
+    <origin xyz="-0.032 0 ${chasis_height}" rpy="0 0 0"/>
   </joint>
   <link name="imu_link"/>
   <joint name="scan_joint" type="fixed">
-    <parent link="link_chassis"/>
+    <parent link="base_link"/>
     <child link="base_scan"/>
-    <origin xyz="-0.032 0 0.172" rpy="0 0 0"/>
+    <origin xyz="0 0 ${chasis_height-0.035}" rpy="0 0 0"/>
   </joint>
   <link name="base_scan">
@@ -185,5 +186,5 @@
     </visual>
     <collision>
-      <origin xyz="0.015 0 -0.0065" rpy="0 0 0"/>
+      <origin xyz="0 0 ${chasis_height}" rpy="0 0 0"/>
       <geometry>
         <cylinder length="0.0315" radius="0.055"/>
@@ -199,10 +200,39 @@
   </link>
   <!-- Gazebo side -->
+  <!--
+  <gazebo reference="wheel_left_link">
+    <mu1>0</mu1>
+    <mu2>0</mu2>
+    <kp>500000.0</kp>
+    <kd>10.0</kd>
+    <minDepth>0.001</minDepth>
+    <maxVel>10</maxVel>
+    <fdir1>1 0 0</fdir1>
+    <material>Gazebo/FlatBlack</material>
+  </gazebo>
+  <gazebo reference="wheel_right_link">
+    <mu1>0</mu1>
+    <mu2>0</mu2>
+    <kp>500000.0</kp>
+    <kd>10.0</kd>
+    <minDepth>0.001</minDepth>
+    <maxVel>10</maxVel>
+    <fdir1>1 0 0</fdir1>
+    <material>Gazebo/FlatBlack</material>
+  </gazebo> -->
+  <gazebo reference="imu_link">
+    <sensor type="imu" name="imu">
+      <always_on>true</always_on>
+      <visualize>$(arg imu_visual)</visualize>
+    </sensor>
+    <material>Gazebo/FlatBlack</material>
+  </gazebo>
   <gazebo>
     <plugin name="kamu_robotu_controller" filename="libgazebo_ros_diff_drive.so">
+      <legacyMode>false</legacyMode>
       <alwaysOn>true</alwaysOn>
       <updateRate>20</updateRate>
-      <leftJoint>joint_left_wheel</leftJoint>
-      <rightJoint>joint_right_wheel</rightJoint>
+      <leftJoint>wheel_left_joint</leftJoint>
+      <rightJoint>wheel_right_joint</rightJoint>
       <wheelSeparation>0.2</wheelSeparation>
       <wheelDiameter>0.48</wheelDiameter>
@@ -211,5 +241,5 @@
       <odometryTopic>odom</odometryTopic>
       <odometryFrame>odom</odometryFrame>
-      <robotBaseFrame>link_chassis</robotBaseFrame>
+      <robotBaseFrame>base_link</robotBaseFrame>
     </plugin>
   </gazebo>
@@ -265,5 +295,5 @@
           <type>gaussian</type>
           <mean>0.0</mean>
-          <stddev>0.00</stddev>
+          <stddev>4e-3</stddev>
         </noise>
       </ray>
@@ -274,3 +304,4 @@
     </sensor>
   </gazebo>
+  -->
 </robot>

Commit message: meshes folders under kamu_robotu_gazebo package merged into one

File: ros_ws/src/kamu_robotu/kamu_robotu_gazebo/urdf/kamu_robotu.xacro (robot description, xacro)
@@ -57,5 +57,5 @@
       <origin rpy="0 0 0" xyz="0 0 0"/>
       <geometry>
-        <mesh filename="package://kamu_robotu_gazebo/meshes/base.STL" scale="1 1 1"/>
+        <mesh filename="package://kamu_robotu_gazebo/models/meshes/base.STL" scale="1 1 1"/>
       </geometry>
       <material name="blue"/>

Commit message: hector slam working with the new model, with small problems that needs to be corrected. there is jumps between tf frames, wheel transformations ara not parsed into map etc.

File: ros_ws/src/kamu_robotu/kamu_robotu_gazebo/urdf/kamu_robotu.xacro (robot description, xacro)
@@ -50,5 +50,5 @@
     <collision name="collision_chassis">
       <geometry>
-        <cylinder length="0.015" radius="0.2"/>
+        <cylinder length="0.015" radius="0.1"/>
       </geometry>
     </collision>
@@ -172,4 +172,10 @@
   </joint>
   <link name="imu_link"/>
+  <joint name="base_footprint_joint" type="fixed">
+    <parent link="base_link"/>
+    <child link="base_footprint"/>
+    <origin xyz="0 0 -0.12" rpy="0 0 0"/>
+  </joint>
+  <link name="base_footprint"/>
   <joint name="scan_joint" type="fixed">
     <parent link="base_link"/>

Commit message: both hector_mapping and gmapping works now (for kamu_robotu)

File: ros_ws/src/kamu_robotu/kamu_robotu_gazebo/urdf/kamu_robotu.xacro (robot description, xacro)
@@ -179,11 +179,11 @@
   <link name="base_footprint"/>
   <joint name="scan_joint" type="fixed">
-    <parent link="base_link"/>
+    <parent link="base_footprint"/>
     <child link="base_scan"/>
-    <origin xyz="0 0 ${chasis_height-0.035}" rpy="0 0 0"/>
+    <origin xyz="0 0 ${chasis_height+0.085}" rpy="0 0 0"/>
   </joint>
   <link name="base_scan">
     <visual>
-      <origin xyz="0 0 0.0" rpy="0 0 0"/>
+      <origin xyz="0 0 0" rpy="0 0 0"/>
       <geometry>
         <mesh filename="package://turtlebot3_description/meshes/sensors/lds.stl" scale="0.001 0.001 0.001"/>
@@ -192,5 +192,5 @@
     </visual>
     <collision>
-      <origin xyz="0 0 ${chasis_height}" rpy="0 0 0"/>
+      <origin xyz="0 0 0" rpy="0 0 0"/>
       <geometry>
         <cylinder length="0.0315" radius="0.055"/>
@@ -281,5 +281,5 @@
     <material>Gazebo/FlatBlack</material>
     <sensor type="ray" name="lds_lfcd_sensor">
-      <pose>0 0 0 0 0 0</pose>
+      <pose>0 0 -0.2 0 0 0</pose>
       <visualize>$(arg laser_visual)</visualize>
       <update_rate>2</update_rate>

Commit message: Now we can choose which robot to spawn while launching maps using robot:=kamu_robotu or robot:=turtlebot3 as argument

File: ros_ws/src/kamu_robotu/kamu_robotu_gazebo/urdf/kamu_robotu.xacro (robot description, xacro)
@@ -32,11 +32,11 @@
   </material>
   <gazebo reference="base_link">
-    <material>Gazebo/Orange</material>
+    <material>Gazebo/FlatBlack</material>
   </gazebo>
   <gazebo reference="wheel_left_link">
-    <material>Gazebo/Blue</material>
+    <material>Gazebo/Red</material>
   </gazebo>
   <gazebo reference="wheel_right_link">
-    <material>Gazebo/Blue</material>
+    <material>Gazebo/Red</material>
   </gazebo>
   <link name="base_link">

Commit message: maps updated to be statc so that it wont move. Gmapping parameter delta updated to see better results

File: ros_ws/src/kamu_robotu/kamu_robotu_gazebo/urdf/kamu_robotu.xacro (robot description, xacro)
@@ -44,7 +44,9 @@
     <pose>0 0 0.1 0 0 0</pose>
     <inertial>
-      <mass value="5"/>
+      <mass value="8.2573504e-01"/>
       <origin rpy="0 0 0" xyz="0 0 0.1"/>
-      <inertia ixx="0.0395416666667" ixy="0" ixz="0" iyy="0.106208333333" iyz="0" izz="0.106208333333"/>
+    <inertia ixx="2.2124416e-03" ixy="-1.2294101e-05" ixz="3.4938785e-05"
+               iyy="2.1193702e-03" iyz="-5.0120904e-06"
+               izz="2.0064271e-03" />
     </inertial>
     <collision name="collision_chassis">
@@ -111,7 +113,9 @@
   <link name="wheel_right_link">
     <inertial>
-      <mass value="0.2"/>
       <origin rpy="0 1.5707 1.5707" xyz="0 0 0"/>
-      <inertia ixx="0.00052666666" ixy="0" ixz="0" iyy="0.00052666666" iyz="0" izz="0.001"/>
+      <mass value="2.8498940e-02" />
+      <inertia ixx="1.1175580e-05" ixy="-4.2369783e-11" ixz="-5.9381719e-09"
+               iyy="1.1192413e-05" iyz="-1.4400107e-11"
+               izz="2.0712558e-05" />
     </inertial>
     <collision name="wheel_right_link_collision">
@@ -131,7 +135,9 @@
   <link name="wheel_left_link">
     <inertial>
-      <mass value="0.2"/>
       <origin rpy="0 1.5707 1.5707" xyz="0 0 0"/>
-      <inertia ixx="0.00052666666" ixy="0" ixz="0" iyy="0.00052666666" iyz="0" izz="0.001"/>
+      <mass value="2.8498940e-02" />
+      <inertia ixx="1.1175580e-05" ixy="-4.2369783e-11" ixz="-5.9381719e-09"
+               iyy="1.1192413e-05" iyz="-1.4400107e-11"
+               izz="2.0712558e-05" />
     </inertial>
     <collision name="wheel_left_link_collision">
@@ -243,5 +249,6 @@
       <wheelSeparation>0.2</wheelSeparation>
       <wheelDiameter>0.048</wheelDiameter>
-      <torque>0.1</torque>
+      <wheelAcceleration>1</wheelAcceleration>
+      <wheelTorque>10</wheelTorque>
       <commandTopic>cmd_vel</commandTopic>
       <odometryTopic>odom</odometryTopic>
@@ -301,5 +308,5 @@
           <type>gaussian</type>
           <mean>0.0</mean>
-          <stddev>4e-3</stddev>
+          <stddev>4e-4</stddev>
         </noise>
       </ray>

File: ros_ws/src/turtlebot3/turtlebot3_description/urdf/turtlebot3_burger.gazebo.xacro (robot description, xacro)
@@ -97,9 +97,9 @@
       <pose>0 0 0 0 0 0</pose>
       <visualize>$(arg laser_visual)</visualize>
-      <update_rate>2</update_rate>
+      <update_rate>5</update_rate>
       <ray>
         <scan>
           <horizontal>
-            <samples>64</samples>
+            <samples>360</samples>
             <resolution>1</resolution>
             <min_angle>0.0</min_angle>

Commit message: Kamurobotu xacro updated, new maps added, carto tutorial updated

File: ros_ws/src/kamu_robotu/kamu_robotu_gazebo/urdf/kamu_robotu.xacro (robot description, xacro)
@@ -193,5 +193,5 @@
       <origin xyz="0 0 0" rpy="0 0 0"/>
       <geometry>
-        <mesh filename="package://turtlebot3_description/meshes/sensors/lds.stl" scale="0.001 0.001 0.001"/>
+        <cylinder length="0.1" radius="0.1"/>
       </geometry>
       <material name="dark"/>

Commit message: Simulation rotation axes are same as the real robot now, lidar bridge max range changed to 1.2meters, follow wall small mistakes corrected

File: ros_ws/src/kamu_robotu/kamu_robotu_gazebo/urdf/kamu_robotu.xacro (robot description, xacro)
@@ -156,5 +156,5 @@
   <!--   Joint for right wheel  -->
   <joint name="wheel_right_joint" type="continuous">
-    <origin rpy="0 0 0" xyz="0 ${wheel_seperation/2} -${chasis_height/2}"/>
+    <origin rpy="0 0 0" xyz="0 -${wheel_seperation/2} -${chasis_height/2}"/>
     <child link="wheel_right_link" />
     <parent link="base_link"/>
@@ -165,5 +165,5 @@
   <!--   Joint for left wheel  -->
   <joint name="wheel_left_joint" type="continuous">
-    <origin rpy="0 0 0" xyz="0 -${wheel_seperation/2} -${chasis_height/2}"/>
+    <origin rpy="0 0 0" xyz="0 ${wheel_seperation/2} -${chasis_height/2}"/>
     <child link="wheel_left_link" />
     <parent link="base_link"/>
@@ -301,6 +301,6 @@
         </scan>
         <range>
-          <min>0.12</min>
-          <max>3.5</max>
+          <min>0.092</min>
+          <max>1.2</max>
           <resolution>0.02</resolution>
         </range>
@@ -308,5 +308,5 @@
           <type>gaussian</type>
           <mean>0.0</mean>
-          <stddev>4e-4</stddev>
+          <stddev>6e-3</stddev>
         </noise>
       </ray>

Commit message: Xacro parameters updated according to real robot, follow wall is now waiting 20 seconds beforehand

File: ros_ws/src/kamu_robotu/kamu_robotu_gazebo/urdf/kamu_robotu.xacro (robot description, xacro)
@@ -3,7 +3,7 @@
   <xacro:arg name="laser_visual" default="false"/>
   <xacro:arg name="imu_visual"   default="false"/>
-  <xacro:property name="wheel_radius" value="0.024" />
+  <xacro:property name="wheel_radius" value="0.02634" />
   <xacro:property name="wheel_length" value="0.01" />
-  <xacro:property name="wheel_seperation" value="0.2" />
+  <xacro:property name="wheel_seperation" value="0.192" />
   <xacro:property name="chasis_height" value="0.115" />
   <material name="black">
@@ -156,5 +156,5 @@
   <!--   Joint for right wheel  -->
   <joint name="wheel_right_joint" type="continuous">
-    <origin rpy="0 0 0" xyz="0 -${wheel_seperation/2} -${chasis_height/2}"/>
+    <origin rpy="0 0 0" xyz="0 ${wheel_seperation/2} -${chasis_height/2}"/>
     <child link="wheel_right_link" />
     <parent link="base_link"/>
@@ -165,5 +165,5 @@
   <!--   Joint for left wheel  -->
   <joint name="wheel_left_joint" type="continuous">
-    <origin rpy="0 0 0" xyz="0 ${wheel_seperation/2} -${chasis_height/2}"/>
+    <origin rpy="0 0 0" xyz="0 -${wheel_seperation/2} -${chasis_height/2}"/>
     <child link="wheel_left_link" />
     <parent link="base_link"/>
